Commit message: script 두개 작성

File: prius_description/urdf/prius.urdf (robot description, URDF)
Before this commit: robot prius, 24 links, 23 joints
Links:
- removed link back_left_far_sonar_link
- removed link back_left_middle_sonar_link
- removed link back_right_far_sonar_link
- removed link back_right_middle_sonar_link
- removed link center_laser_link
- removed link front_left_far_sonar_link
- removed link front_left_laser_link
- removed link front_left_middle_sonar_link
- removed link front_right_far_sonar_link
- removed link front_right_laser_link
- removed link front_right_middle_sonar_link
- added link velodyne_center_link, mass 1
- added link velodyne_front_left_link, mass 1
- added link velodyne_front_right_link, mass 1
Joints:
- removed joint back_left_far_sonar_joint
- removed joint back_left_middle_sonar_joint
- removed joint back_right_far_sonar_joint
- removed joint back_right_middle_sonar_joint
- removed joint center_laser_joint
- removed joint front_left_far_sonar_joint
- removed joint front_left_laser_joint
- removed joint front_left_middle_sonar_joint
- removed joint front_right_far_sonar_joint
- removed joint front_right_laser_joint
- removed joint front_right_middle_sonar_joint
- added joint velodyne_center_joint: type fixed, parent chassis, child velodyne_center_link, origin xyz=0 0.4 1.8 rpy=0 0 -1.5707
- added joint velodyne_front_left_joint: type fixed, parent chassis, child velodyne_front_left_link, origin xyz=1 -2.3 0.5 rpy=0 0.05 0
- added joint velodyne_front_right_joint: type fixed, parent chassis, child velodyne_front_right_link, origin xyz=-1 -2.3 0.5 rpy=0 0.05 3.14

Commit message: mapping 완성, matching수행해야됨

File: prius_description/urdf/prius.urdf (robot description, URDF)
Before this commit: robot prius, 16 links, 15 joints
Links:
- removed link velodyne_center_link
- added link velodyne, mass 1
Joints:
- removed joint velodyne_center_joint
- added joint velodyne: type fixed, parent chassis, child velodyne, origin xyz=0 0.4 1.8 rpy=0 0 -1.5707
